Commit message: Drawing dish bin envs and some model syncing

File: models/dish_models/mug_1_decomp/mug_1_decomp.urdf (robot description, URDF)
Before this commit: robot plate_11in_decomp, 1 links, 0 joints
Links:
- removed link plate_11in_decomp_body_link
- added link mug_1_decomp_body_link, mass 2.00E-01; collision mesh filename=mug_1_decomp_convex_piece_0.obj scale=1.0000E+00 1.0000E+00 1.0000E+00; collision mesh filename=mug_1_decomp_convex_piece_1.obj scale=1.0000E+00 1.0000E+00 1.0000E+00

File: models/dish_models/mug_2_decomp/mug_2_decomp.urdf (robot description, URDF)
Before this commit: robot plate_11in_decomp, 1 links, 0 joints
Links:
- removed link plate_11in_decomp_body_link
- added link mug_2_decomp_body_link, mass 2.00E-01; collision mesh filename=mug_2_decomp_convex_piece_0.obj scale=1.0000E+00 1.0000E+00 1.0000E+00; collision mesh filename=mug_2_decomp_convex_piece_1.obj scale=1.0000E+00 1.0000E+00 1.0000E+00
